File: PCB/Plant_Thing.kicad_pcb (KiCad board)
At the start: 2 copper layers, 40 x 60 mm, 89 parts, among them IC1 NCP333FCT2G, IC2 NCP333FCT2G, IC3 NCP333FCT2G, J1 Conn_ARM_SWD_TagConnect_TC203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, J3 Conn_Coaxial_Small, J4 Conn_01x03_Socket, Q1 NMOS, Q2 NMOS, U1 nRF52820-QDxx, U2 BQ297xy, U3 BQ24090DGQ, U4 LTR-303ALS-01, U5 TLC59283RGER, U6 TPS63001, Y1 32M

Commit message: Continued on Devboard
Parts:
- removed J4: Conn_01x03_Socket, Connector_PinSocket_2.54mm:PinSocket_1x03_P2.54mm_Horizontal
- added C33: 100n, Capacitor_SMD:C_0402_1005Metric, F.Cu at (169.7, 92.7)
- added J2: LED, Connector_PinHeader_2.54mm:PinHeader_1x02_P2.54mm_Vertical, F.Cu at (171.5, 84.2)
- added J6: TDT, Connector_PinHeader_2.54mm:PinHeader_1x02_P2.54mm_Vertical, F.Cu at (158.8, 65.9)
- added J7: VDDH, Connector_PinHeader_2.54mm:PinHeader_1x02_P2.54mm_Vertical, F.Cu at (132.2, 91.9)
- added J8: EXT 3.3V, Connector_PinHeader_2.54mm:PinHeader_1x02_P2.54mm_Vertical, F.Cu at (165.5, 117.8)
- added JP1: SolderJumper_3_Bridged12, Jumper:SolderJumper-3_P1.3mm_Bridged12_RoundedPad1.0x1.5mm, F.Cu at (159.7, 97.7)
- added JP2: SolderJumper_3_Bridged12, Jumper:SolderJumper-3_P1.3mm_Bridged12_RoundedPad1.0x1.5mm, F.Cu at (159.7, 95.0)
- added JP3: SolderJumper_3_Bridged12, Jumper:SolderJumper-3_P1.3mm_Bridged12_RoundedPad1.0x1.5mm, F.Cu at (136.7, 91.4)
- added R11: 5k1, Resistor_SMD:R_0402_1005Metric, F.Cu at (95.3, 103.9)
- added R12: 5k1, Resistor_SMD:R_0402_1005Metric, F.Cu at (95.3, 105.9)
- added R13: 5k3, Resistor_SMD:R_0402_1005Metric, F.Cu at (167.2, 92.1)
- added SW1: MK-12C02-G020, G-Switch:SW-SMD_MK-12C02-G020, F.Cu at (142.5, 117.5)
- added TP10: TestPoint_Small, TestPoint:TestPoint_Pad_D1.0mm, F.Cu at (169.0, 95.0)
- added TP11: TestPoint_Small, TestPoint:TestPoint_Pad_D1.0mm, F.Cu at (173.1, 95.8)
- added TP12: TestPoint_Small, TestPoint:TestPoint_Pad_D1.0mm, F.Cu at (167.8, 90.3)
- added TP13: TestPoint_Small, TestPoint:TestPoint_Pad_D1.0mm, F.Cu at (172.2, 63.4)
- added TP8: TestPoint_Small, TestPoint:TestPoint_Pad_D1.0mm, F.Cu at (69.6, 110.9)
- added TP9: TestPoint_Small, TestPoint:TestPoint_Pad_D1.0mm, F.Cu at (171.0, 95.6)
- added U7: SRV05-4, Package_TO_SOT_SMD:SOT-23-6, F.Cu at (155.0, 109.0)
- added X1: HY32768KSMD3068YA2R30, HY32768KSMD3068YA2R30:CRYSTAL-SMD_L7.0-W3.2-LS7.5, F.Cu at (159.8, 87.1)
- AE1: value Antenna -> Antenna_Shield; footprint RF_Antenna:Texas_SWRA117D_2.4GHz_Right -> RF_Antenna:Texas_SWRA117D_2.4GHz_Left
- J3: value Conn_Coaxial_Small -> Conn_01x06_Pin; footprint Connector_Coaxial:U.FL_Molex_MCRF_73412-0110_Vertical -> Connector_PinHeader_2.54mm:PinHeader_1x06_P2.54mm_Vertical
- moved C8 112.3 mm to (170.8, 117.9), turned to 90 degrees
- moved C4 93.9 mm to (162.2, 73.3), turned to 180 degrees
- moved C1 87.1 mm to (156.5, 82.5), turned to 90 degrees
- moved C16 86.8 mm to (162.4, 84.7), turned to 180 degrees
- moved C17 81.1 mm to (157.1, 84.7)
- moved R4 80.0 mm to (66.6, 94.6)
- moved C2 77.9 mm to (149.6, 73.7)
- moved TP1 74.7 mm to (155.0, 70.7)
- moved R1 71.5 mm to (66.6, 88.6)
- moved R2 71.3 mm to (66.6, 90.6)
- moved R3 71.2 mm to (66.6, 92.6), turned to 0 degrees
- moved R5 70.8 mm to (66.6, 96.6)
- moved TP6 69.2 mm to (69.6, 107.8)
- moved U4 68.9 mm to (169.1, 62.4), turned to 180 degrees
- moved R6 67.7 mm to (66.6, 98.6), turned to 0 degrees
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Connections:
- net Net-(SW1-B) renamed VCC
- AE1 pad 2: (no net) -> GND
- C25 pad 1: Net-(U6-EN) -> /Power/VINA
- C26 pad 1: Net-(U6-FB) -> +3.3V
- C27 pad 1: Net-(U6-FB) -> +3.3V
- C28 pad 1: Net-(U6-FB) -> +3.3V
- C29 pad 1: unconnected-(C29-Pad1) -> +3.3V
- C29 pad 2: unconnected-(C29-Pad2) -> GND
- C30 pad 1: unconnected-(C30-Pad1) -> VDDA
- C30 pad 2: unconnected-(C30-Pad2) -> GND
- C31 pad 1: Net-(IC3-IN) -> +3.3V
- D1 pad 2: unconnected-(D1-A-Pad2) -> Net-(D1-A)
- D10 pad 2: unconnected-(D10-A-Pad2) -> Net-(D1-A)
- D11 pad 2: unconnected-(D11-A-Pad2) -> Net-(D1-A)
- D12 pad 2: unconnected-(D12-A-Pad2) -> Net-(D1-A)
- D13 pad 2: unconnected-(D13-A-Pad2) -> Net-(D1-A)
- D14 pad 2: unconnected-(D14-A-Pad2) -> Net-(D1-A)
- D2 pad 2: unconnected-(D2-A-Pad2) -> Net-(D1-A)
- D3 pad 2: unconnected-(D3-A-Pad2) -> Net-(D1-A)
- D4 pad 2: unconnected-(D4-A-Pad2) -> Net-(D1-A)
- D5 pad 2: unconnected-(D5-A-Pad2) -> Net-(D1-A)
- D6 pad 2: unconnected-(D6-A-Pad2) -> Net-(D1-A)
- D7 pad 2: unconnected-(D7-A-Pad2) -> Net-(D1-A)
- D8 pad 2: unconnected-(D8-A-Pad2) -> Net-(D1-A)
- D9 pad 2: unconnected-(D9-A-Pad2) -> Net-(D1-A)
- IC2 pad A1: unconnected-(IC2-OUT-PadA1) -> VDDA
- IC2 pad A2: unconnected-(IC2-IN-PadA2) -> +3.3V
- IC2 pad B1: unconnected-(IC2-GND-PadB1) -> GND
- IC2 pad B2: unconnected-(IC2-EN-PadB2) -> P0.07_EN_SENSOR_BUS
- IC3 pad A2: Net-(IC3-IN) -> +3.3V
- J3 pad 1: unconnected-(J3-In-Pad1) -> GND
- J3 pad 2: unconnected-(J3-Ext-Pad2) -> P0.03_TDT_MEASURE
- R10 pad 2: Net-(U6-EN) -> /Power/VINA
- TP3 pad 1: +BATT -> P0.14_SCL
- TP4 pad 1: -BATT -> P0.15_SDA
- U1 pad 4: unconnected-(U1-AIN2/P0.04-Pad4) -> P0.04_AGPIO
- U1 pad 5: unconnected-(U1-AIN3/P0.05-Pad5) -> P0.05_EN_DCDC
- U1 pad 9: VDD -> /VDDH
- U4 pad 5: unconnected-(U4-INT-Pad5) -> Net-(U4-INT)
- U5 pad 20: unconnected-(U5-IREF-Pad20) -> Net-(U5-IREF)
- U5 pad 21: Net-(IC3-OUT) -> Net-(D1-A)
- U6 pad 1: Net-(U6-FB) -> +3.3V
- U6 pad 10: Net-(U6-FB) -> +3.3V
- U6 pad 6: Net-(U6-EN) -> /Power/EN
- U6 pad 7: unconnected-(U6-PS/SYNC-Pad7) -> /Power/PS
- U6 pad 8: Net-(U6-EN) -> /Power/VINA
- USB1 pad 1: unconnected-(USB1-GND-Pad1) -> GND
- USB1 pad 10: unconnected-(USB1-CC2-Pad10) -> Net-(USB1-CC2)
- USB1 pad 11: unconnected-(USB1-VBUS-Pad11) -> VBUS
- USB1 pad 12: unconnected-(USB1-GND-Pad12) -> GND
- USB1 pad 13: unconnected-(USB1-SHELL-Pad13) -> GND
- USB1 pad 14: unconnected-(USB1-SHELL-Pad14) -> GND
- USB1 pad 2: unconnected-(USB1-VBUS-Pad2) -> VBUS
- USB1 pad 4: unconnected-(USB1-CC1-Pad4) -> Net-(USB1-CC1)
- USB1 pad 5: unconnected-(USB1-DN2-Pad5) -> Net-(U7-IO2)
- USB1 pad 6: unconnected-(USB1-DP1-Pad6) -> Net-(U7-IO1)
- USB1 pad 7: unconnected-(USB1-DN1-Pad7) -> Net-(U7-IO2)
- USB1 pad 8: unconnected-(USB1-DP2-Pad8) -> Net-(U7-IO1)
Routing:
- net Net-(D1-A): track 0.00 -> 94.5 mm, vias 0 -> 8
- net P0.28_LAT: track 0.00 -> 43.3 mm, vias 0 -> 2
- net P0.29_SCLK: track 0.00 -> 41.7 mm, vias 0 -> 2
- net USB_DN: track 0.00 -> 40.9 mm, vias 0 -> 2
- net P0.30_SIN: track 0.00 -> 39.6 mm, vias 0 -> 2
- net USB_DP: track 0.00 -> 38.7 mm, vias 0 -> 2
- net P0.08_EN_LED: track 4.77 -> 39.9 mm, vias 0 -> 4
- net P0.20_BLANK: track 0.00 -> 34.7 mm, vias 0 -> 2
- net SWDIO: track 0.00 -> 25.5 mm, vias 0 -> 2
- net P0.18_RESET: track 0.00 -> 24.8 mm
- net P0.05_EN_DCDC: track 0.00 -> 24.4 mm, vias 0 -> 2
- net SWDCLK: track 0.00 -> 24.2 mm, vias 0 -> 2
- net P0.14_SCL: track 0.00 -> 20.5 mm, vias 0 -> 2
- net P0.07_EN_SENSOR_BUS: track 0.00 -> 20.1 mm
- net P0.15_SDA: track 0.00 -> 18.7 mm
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- added copper zone on B.Cu, net GND
- added copper zone on F.Cu, net GND
- added copper zone on In1.Cu, net GND
- added copper zone on In2.Cu, net GND
Other:
- board size 40 x 60 mm -> 50 x 60 mm
- copper layers 2 -> 4
- board text removed: "LED BAR"
- board text removed: "POWER"
- board text removed: "SENSE"
- board text removed: "nRF52820"
