File: PCB/io.kicad_sch (KiCad schematic)
At the start: 31 parts, among them IC3 NCP333FCT2G, J1 Conn_ARM_SWD_TagConnect_TC203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, J2 LED, U5 TLC59283RGER, U7 SRV05-4

Commit message: Finished Devboard
Parts:
- removed C31, C32: 100n, Capacitor_SMD:C_0402_1005Metric, symbol Device:C_Small
- removed IC3: NCP333FCT2G, BGA4C40P2X2_76X76X63, symbol NCP333FCT2G:NCP333FCT2G
- removed TP7: TestPoint_Small, TestPoint:TestPoint_Pad_D1.0mm, symbol Connector:TestPoint_Small
Connections:
- net +3.3V: now also J2.2 (Pin_2)
- net USB_DN: now also U7.3 (IO2), USB1.5 (DN2), USB1.7 (DN1); no longer U7.6 (IO4)
- net USB_DP: now also U7.1 (IO1), USB1.6 (DP1), USB1.8 (DP2); no longer U7.4 (IO3)
- no-connect marks 4 -> 6
