File: PCB/power.kicad_sch (KiCad schematic)
At the start: 33 parts, among them IC1 NCP333FCT2G, Q1 NMOS, Q2 NMOS, SW1 MK-12C02-G020, U2 BQ297xy, U3 BQ24090DGQ, U6 TPS63001

Commit message: Finished Devboard
Parts:
- added D15: LED_Small, LED_SMD:LED_0805_2012Metric, symbol Device:LED_Small
- added R14, R15: 10k, Resistor_SMD:R_0402_1005Metric, symbol Device:R_Small
- C28: value 10u -> 330u; footprint Capacitor_SMD:CP_Elec_5x4.4 -> Capacitor_SMD:CP_Elec_10x10
- R6: value 300 -> 30k
- R7: value 1k1 -> 110k
Connections:
- net +BATT: now also R14.2, R15.2
- net P0.16_CHG: now also D15.2 (A), R14.1; no longer U3.8 (~{CHG})
- net P0.17_PG: now also R15.1
- net P0.05_EN_DCDC renamed P0.08_EN_DCDC
- new net: D15.1 (K), U3.8 (~{CHG})
Other:
- note removed: "TODO: pull up/down for CHG and PG"
